File: MicropendousX/Hardware/MicropendousX-176x/MicropendousX-176x.sch (KiCad schematic (older format))
At the start: 219 parts, among them IC1 LPC176X, IC2 AP2101, IC4 LAN8720, IC5 TS3USB221, J1 PULSE_J0011_PHY_SIDE, P8 Bottom, P9 Top, Q1 PCH, SW1 RESET, SW2 NMI, U1 USB-miniB, U2 USB-A, U3 CONN_MICROSD, U4 1117-3.3, U6 JTAG, X1 12MHz, X2 32.768kHz, X3 25MHz

Commit message: Updated LPC176x hardware design with top layer silkcreen pin names and minor fixes for copper layers.
Parts:
- C1, C2: value 33pF -> 33p
- C10, C11, C8, C9: value 12pF -> 12p
- C12, C16: value 1uF -> 1u
- C13, C17, C19, C21, C24, C41: value 10uF -> 10u
- C18, C20, C22, C25, C26, C28, C29, C30, C36, C37, C38, C39, C7: value 0.1uF -> 0u1
- C23: value 0.01uF -> u01
- C3, C4, C5, C6: value 22pF -> 22p
- C35: value 120uF -> 120u
- C40: value 33uF -> 33u
- CR1, CR2: value ESD_ZENER -> ESD
- R13: value 12.1k -> 12k1
- R23: value 4.7k -> 4k7
- R33: value 1.5k -> 1k5
Connections:
- wire segments 330 -> 383
Other:
- note removed: "DNI-Test Only"

Commit message: Updated MicropendousX-176x to a better stocked microSD connector (Amphenol 101-00303).
Parts:
- added C42: 0u1, symbol C_MINI
- U3: value CONN_MICROSD -> microSD
Changed lines of the file:
@@
-EESchema Schematic File Version 2  date 12/10/2010 22:28:42
+EESchema Schematic File Version 2  date 13/10/2010 07:56:43
 LIBS:power
 LIBS:device
@@
 Comment4 "www.MicropendousX.org"
 $EndDescr
-$Comp
-L GND #PWR01
-U 1 1 4CB51801
-P 7450 8050
-F 0 "#PWR01" H 7450 8050 30  0001 C CNN
-F 1 "GND" H 7450 7980 30  0001 C CNN
-	1    7450 8050
-	1    0    0    -1
-$EndComp
+Connection ~ 4800 7050
+Wire Wire Line
+	4950 7050 4350 7050
 Wire Wire Line
 	7450 8050 7450 7900
@@
 Connection ~ 4500 7050
 Connection ~ 4500 6850
-Wire Wire Line
-	4800 7050 4350 7050
 Connection ~ 11050 8200
 Wire Wire Line
@@
 	900  5950 900  6000
 Wire Wire Line
-	4800 6850 4350 6850
-Wire Wire Line
 	5400 1750 5400 2850
 Wire Wire Line
@@
 Wire Wire Line
 	3450 1350 3450 1400
+Wire Wire Line
+	4950 6850 4350 6850
+Connection ~ 4800 6850
+$Comp
+L C_MINI C42
+U 1 1 4CB59E4B
+P 4950 6950
+F 0 "C42" V 4900 7000 30  0000 C CNN
+F 1 "0u1" V 5000 7000 25  0000 C CNN
+	1    4950 6950
+	0    1    1    0
+$EndComp
+$Comp
+L GND #PWR01
+U 1 1 4CB51801
+P 7450 8050
+F 0 "#PWR01" H 7450 8050 30  0001 C CNN
+F 1 "GND" H 7450 7980 30  0001 C CNN
+	1    7450 8050
+	1    0    0    -1
+$EndComp
 Text Label 3450 1000 0    20   ~ 0
 2DN
@@
 P 1000 1450
 F 0 "U3" H 825 1025 40  0000 C CNN
-F 1 "CONN_MICROSD" H 1050 2000 30  0000 C CNN
+F 1 "microSD" H 1050 2000 30  0000 C CNN
 	1    1000 1450
 	-1   0    0    -1
